Commit message: refactor(ur10/calibration): simplify XML/URDF export logic and remove verbose logging
- Remove Apache 2.0 license header and unused imports (time, __future__)
- Simplify export_xml() and export_urdf_dynamics() by assuming all required keys exist in input dicts
  - Replace body_map.get() with direct dict access (body_map[target])
  - Remove None-checks and early-continue branches for missing bodies/joints
  - Remove verbose logging statements for each updated element
- Remove redundant _get_body()

File: models/ur_description/urdf/ur10_robot.urdf (robot description, URDF)
Before this commit: robot ur10, 11 links, 10 joints
Links:
- link forearm_link: mass 3.87 -> 3.870025432
- link shoulder_link: mass 7.778 -> 7.778002758
- link upper_arm_link: mass 12.93 -> 12.93000254
- link wrist_1_link: mass 1.96 -> 1.960005271
- link wrist_2_link: mass 1.96 -> 1.960005271
- link wrist_3_link: mass 0.202 -> 0.2019997562
